File: Mezzanine_Board.kicad_pcb (KiCad board)
At the start: 2 copper layers, 8 parts, among them P1 CONN_02X50, P2 CONN_02X50, P3 CONN_02X50, P4 CONN_02X50

Commit message: Add files via upload
Parts:
- removed the REF** at (85.1, 55.9)
- removed the REF** at (158.8, 55.9)
- removed the REF** at (81.3, 141.6)
- removed the REF** at (161.3, 141.6)
- added P7: CONN_02X30, Connectors_Samtec:MECF-30-0_-NP-L-DV_Edge, F.Cu at (120.6, 165.1)
- added REF**: MountingHole_3.2mm_M3_Pad, Mounting_Holes:MountingHole_3.2mm_M3_Pad, F.Cu at (93.6, 67.3)
- added REF**: MountingHole_3.2mm_M3_Pad, Mounting_Holes:MountingHole_3.2mm_M3_Pad, F.Cu at (147.6, 67.3)
- added REF**: MountingHole_3.2mm_M3_Pad, Mounting_Holes:MountingHole_3.2mm_M3_Pad, F.Cu at (93.6, 159.3)
- added REF**: MountingHole_3.2mm_M3_Pad, Mounting_Holes:MountingHole_3.2mm_M3_Pad, F.Cu at (147.6, 159.3)
Connections:
- P1 pad 1: Net-(P1-Pad100) -> /JTAG_TMS
- P1 pad 10: /RSTN_C2M -> /HDMI_PD
- P1 pad 100: /HDMI_D23 -> Net-(P1-Pad100)
- P1 pad 11: GND -> /CAM_DATA2_P
- P1 pad 12: /PWR_ENABLE -> /CAM_DATA1_P
- P1 pad 13: /SFP_GBT_RX_N -> /CAM_DATA2_N
- P1 pad 14: /CFG_DONE -> /CAM_DATA1_N
- P1 pad 15: /MGTRX2_N -> GND
- P1 pad 16: /CFG_VBATT -> GND
- P1 pad 17: /SFP_GBT_RX_P -> /CAM_DATA4_P
- P1 pad 18: /HDMI_INTN -> /CAM_DATA3_P
- P1 pad 19: /MGTRX2_P -> /CAM_DATA4_N
- P1 pad 20: /HDMI_PD -> /CAM_DATA3_N
- P1 pad 21: /FMC_GBT_REFCLK_N -> GND
- P1 pad 22: /CAM_DATA2_P -> GND
- P1 pad 23: /FMC_GBT_RX_N -> /CAM_DATA6_P
- P1 pad 24: /CAM_DATA1_P -> /CAM_DATA5_P
- P1 pad 25: /FMC_GBT_REFCLK_P -> /CAM_DATA6_N
- P1 pad 26: /CAM_DATA2_N -> /CAM_DATA5_N
- P1 pad 27: /FMC_GBT_RX_P -> GND
- P1 pad 28: /CAM_DATA1_N -> GND
- P1 pad 29: GND -> /CAM_SPI_EN
- P1 pad 3: Net-(P1-Pad99) -> /FPGA_TDI
- P1 pad 30: GND -> /CAM_DATA7_P
- P1 pad 31: GND -> /CAM_SPI_CLK
- P1 pad 32: GND -> /CAM_DATA7_N
- P1 pad 33: /PB_GPIO_0 -> GND
- P1 pad 34: /CAM_DATA4_P -> GND
- P1 pad 35: /CAM_CLK_N -> /CAM_SPI_MISO
- P1 pad 36: /CAM_DATA3_P -> /HDMI_SPDIF
- P1 pad 37: /CAM_REFCLK -> /CAM_SPI_MOSI
- P1 pad 38: /CAM_DATA4_N -> /HDMI_SPDIF_OUT
- P1 pad 39: /CAM_CLK_P -> GND
- P1 pad 4: /JTAG_TCK -> /FPGA_TDO
- P1 pad 40: /CAM_DATA3_N -> GND
- P1 pad 41: /VADJ -> /HDMI_D20
- P1 pad 42: GND -> /HDMI_VSYNC
- P1 pad 43: /VADJ -> /HDMI_D21
- P1 pad 44: GND -> /HDMI_HSYNC
- P1 pad 46: /CAM_DATA6_P -> GND
- P1 pad 47: /VADJ -> /CAM_SYNC_P
- P1 pad 48: /CAM_DATA5_P -> /HDMI_D22
- P1 pad 49: /HDMI_D35 -> /CAM_SYNC_N
- P1 pad 5: Net-(P1-Pad98) -> /RSTN_C2M
- P1 pad 50: /CAM_DATA6_N -> /HDMI_D23
- P1 pad 51: /HDMI_DE -> GND
- P1 pad 52: /CAM_DATA5_N -> GND
- P1 pad 53: /HDMI_D34 -> /HDMI_D24
- P1 pad 54: GND -> /CAM_DATA0_P
- P1 pad 55: /HDMI_CLK -> /HDMI_D25
- P1 pad 56: GND -> /CAM_DATA0_N
- P1 pad 57: GND -> /VIN_HDR
- P1 pad 58: /CAM_SPI_EN -> /VIN_HDR
- P1 pad 59: GND -> /VIN_HDR
- P1 pad 6: /FPGA_TDI -> /PWR_ENABLE
- P1 pad 60: /CAM_DATA7_P -> /VIN_HDR
- P1 pad 61: /HDMI_D31 -> /HDMI_D28
- P1 pad 62: /CAM_SPI_CLK -> /HDMI_D26
- P1 pad 63: /HDMI_D33 -> /HDMI_D29
- P1 pad 64: /CAM_DATA7_N -> /HDMI_D27
- P1 pad 65: /HDMI_D30 -> GND
- P1 pad 68: GND -> /HDMI_D30
- P1 pad 69: GND -> /HDMI_D33
- P1 pad 7: Net-(P1-Pad97) -> /CFG_DONE
- P1 pad 70: /CAM_SPI_MISO -> /HDMI_D31
- P1 pad 72: /HDMI_SPDIF -> GND
- P1 pad 73: /HDMI_D27 -> /HDMI_CLK
- P1 pad 74: /CAM_SPI_MOSI -> /HDMI_D34
- P1 pad 75: /HDMI_D29 -> /HDMI_DE
- P1 pad 76: /HDMI_SPDIF_OUT -> /HDMI_D35
- P1 pad 77: /HDMI_D26 -> /VADJ
- P1 pad 79: /HDMI_D28 -> /VADJ
- P1 pad 8: /FPGA_TDO -> /CFG_VBATT
- P1 pad 80: GND -> /VADJ
- P1 pad 81: /VIN_HDR -> /CAM_CLK_P
- P1 pad 82: /HDMI_D20 -> /CAM_REFCLK
- P1 pad 83: /VIN_HDR -> /CAM_CLK_N
- P1 pad 84: /HDMI_VSYNC -> /PB_GPIO_0
- P1 pad 85: /VIN_HDR -> GND
- P1 pad 86: /HDMI_D21 -> GND
- P1 pad 87: /VIN_HDR -> /FMC_GBT_RX_P
- P1 pad 88: /HDMI_HSYNC -> /FMC_GBT_REFCLK_P
- P1 pad 89: /CAM_DATA0_N -> /FMC_GBT_RX_N
- P1 pad 9: GND -> /HDMI_INTN
- P1 pad 90: GND -> /FMC_GBT_REFCLK_N
- P1 pad 91: /HDMI_D25 -> /MGTRX2_P
- P1 pad 92: GND -> /SFP_GBT_RX_P
- P1 pad 93: /CAM_DATA0_P -> /MGTRX2_N
- P1 pad 94: /CAM_SYNC_P -> /SFP_GBT_RX_N
- P1 pad 95: /HDMI_D24 -> GND
- P1 pad 96: /HDMI_D22 -> GND
- P1 pad 97: GND -> Net-(P1-Pad97)
- P1 pad 98: /CAM_SYNC_N -> Net-(P1-Pad98)
- P1 pad 99: GND -> Net-(P1-Pad99)
- P2 pad 1: /DIP_GPIO_0 -> /FMC_LA20_P
- P2 pad 10: /FMC_LA22_P -> /CFG_INIT__B
- P2 pad 100: /FMC_LA29_N -> /DIP_GPIO_0
- P2 pad 11: /RF_GPIO2_BANK12 -> /VIN_HDR
- P2 pad 12: /FMC_LA21_P -> /PG_MODULE
- P2 pad 13: /SFP_GPIO_4 -> /FMC_PRSNT
- P2 pad 14: /FMC_LA22_N -> /DIP_GPIO_3
- P2 pad 15: /SFP_GPIO_6 -> GND
- P2 pad 16: /FMC_LA21_N -> GND
- P2 pad 17: GND -> /FMC_LA23_P
- P2 pad 18: /VCCIO_EN -> /SCL
- P2 pad 19: GND -> /FMC_LA23_N
- P2 pad 20: Net-(P2-Pad10) -> /SDA
- P2 pad 21: /SFP_GPIO_3 -> GND
- P2 pad 22: /VIN_HDR -> GND
- P2 pad 23: /SFP_GPIO_1 -> /FMC_LA25_P
- P2 pad 24: /PG_MODULE -> /FMC_LA24_P
- P2 pad 25: /SFP_GPIO_2 -> /FMC_LA25_N
- P2 pad 26: /FMC_PRSNT -> /FMC_LA24_N
- P2 pad 27: /SFP_GPIO_0 -> GND
- P2 pad 28: /DIP_GPIO_3 -> GND
- P2 pad 29: GND -> /FMC_LA27_P
- P2 pad 3: Net-(P2-Pad99) -> /FMC_LA20_N
- P2 pad 30: GND -> /FMC_LA26_P
- P2 pad 31: GND -> /FMC_LA27_N
- P2 pad 32: GND -> /FMC_LA26_N
- P2 pad 33: /FMC_LA16_N -> GND
- P2 pad 34: /FMC_LA23_P -> GND
- P2 pad 35: /FMC_LA15_N -> /FMC_LA17_CC_P
- P2 pad 36: /SCL -> /FMC_LA18_CC_P
- P2 pad 37: /FMC_LA16_P -> /FMC_LA17_CC_N
- P2 pad 38: /FMC_LA23_N -> /FMC_LA18_CC_N
- P2 pad 39: /FMC_LA15_P -> GND
- P2 pad 4: /FMC_LA19_P -> /FMC_LA19_N
- P2 pad 40: /SDA -> GND
- P2 pad 41: /1V8 -> /FMC_LA28_P
- P2 pad 42: GND -> /FMC_CLK1_M2C_P
- P2 pad 43: /1V8 -> /FMC_LA28_N
- P2 pad 44: GND -> /FMC_CLK1_M2C_N
- P2 pad 46: /FMC_LA25_P -> GND
- P2 pad 47: /1V8 -> /FMC_LA30_P
- P2 pad 48: /FMC_LA24_P -> /FMC_LA29_P
- P2 pad 49: /I2C3_SCL -> /FMC_LA30_N
- P2 pad 5: /LED_GPIO_3 -> /FMC_LA22_P
- P2 pad 50: /FMC_LA25_N -> /FMC_LA29_N
- P2 pad 51: /SYS_SPI_MOSI -> GND
- P2 pad 52: /FMC_LA24_N -> GND
- P2 pad 53: /I2C3_SDA -> /FMC_LA32_P
- P2 pad 54: GND -> /FMC_LA31_P
- P2 pad 55: /SYS_SPI_SCK -> /FMC_LA32_N
- P2 pad 56: GND -> /FMC_LA31_N
- P2 pad 57: GND -> /VIN_HDR
- P2 pad 58: /FMC_LA27_P -> /VIN_HDR
- P2 pad 59: GND -> /VIN_HDR
- P2 pad 6: /FMC_LA20_N -> /FMC_LA21_P
- P2 pad 60: /FMC_LA26_P -> /VIN_HDR
- P2 pad 61: /I2C2_SCL -> /RF_GPIO0_BANK13
- P2 pad 62: /FMC_LA27_N -> /FMC_LA33_P
- P2 pad 63: /I2C2_SCL -> /RF_GPIO1_BANK13
- P2 pad 64: /FMC_LA26_N -> /FMC_LA33_N
- P2 pad 65: /I2C2_SDA -> GND
- P2 pad 68: GND -> /I2C2_SDA
- P2 pad 69: GND -> /I2C2_SCL
- P2 pad 7: /VADJ -> /FMC_LA22_N
- P2 pad 70: /FMC_LA17_CC_P -> /I2C2_SCL
- P2 pad 72: /FMC_LA18_CC_P -> GND
- P2 pad 73: /FMC_LA33_N -> /SYS_SPI_SCK
- P2 pad 74: /FMC_LA17_CC_N -> /I2C3_SDA
- P2 pad 75: /RF_GPIO1_BANK13 -> /SYS_SPI_MOSI
- P2 pad 76: /FMC_LA18_CC_N -> /I2C3_SCL
- P2 pad 77: /FMC_LA33_P -> /1V8
- P2 pad 79: /RF_GPIO0_BANK13 -> /1V8
- P2 pad 8: /FMC_LA19_N -> /FMC_LA21_N
- P2 pad 80: GND -> /1V8
- P2 pad 81: /VIN_HDR -> /FMC_LA15_P
- P2 pad 82: /FMC_LA28_P -> /FMC_LA16_P
- P2 pad 83: /VIN_HDR -> /FMC_LA15_N
- P2 pad 84: /FMC_CLK1_M2C_P -> /FMC_LA16_N
- P2 pad 85: /VIN_HDR -> GND
- P2 pad 86: /FMC_LA28_N -> GND
- P2 pad 87: /VIN_HDR -> /SFP_GPIO_0
- P2 pad 88: /FMC_CLK1_M2C_N -> /SFP_GPIO_2
- P2 pad 89: /FMC_LA31_N -> /SFP_GPIO_1
- P2 pad 9: /SFP_GPIO_5 -> /VCCIO_EN
- P2 pad 90: GND -> /SFP_GPIO_3
- P2 pad 91: /FMC_LA32_N -> GND
- P2 pad 93: /FMC_LA31_P -> /SFP_GPIO_6
- P2 pad 94: /FMC_LA30_P -> /SFP_GPIO_4
- P2 pad 95: /FMC_LA32_P -> /RF_GPIO2_BANK12
- P2 pad 96: /FMC_LA29_P -> /SFP_GPIO_5
- P2 pad 97: GND -> /VADJ
- P2 pad 98: /FMC_LA30_N -> /LED_GPIO_3
- P2 pad 99: GND -> Net-(P2-Pad99)
- P3 pad 1: /FMC_LA13_N -> /MGTREFCLK1_P
- P3 pad 10: GND -> /1V0_AVCC
- P3 pad 100: GND -> /FMC_LA13_N
- P3 pad 13: /FMC_CLK0_M2C_N -> /MGTTX2_P
- P3 pad 14: /FMC_GBT_TX_P -> /SFP_GBT_TX_P
- P3 pad 15: /FMC_LA12_N -> /MGTTX2_N
- P3 pad 16: /1V0_AVCC -> /SFP_GBT_TX_N
- P3 pad 17: /FMC_CLK0_M2C_P -> GND
- P3 pad 18: /FMC_GBT_TX_N -> GND
- P3 pad 19: /FMC_LA12_P -> /FMC_LA02_P
- P3 pad 20: /1V0_AVCC -> Net-(P3-Pad20)
- P3 pad 21: GND -> /FMC_LA02_N
- P3 pad 22: GND -> Net-(P3-Pad22)
- P3 pad 24: /1V0_AVCC -> GND
- P3 pad 25: /FMC_LA01_CC_N -> /FMC_LA04_P
- P3 pad 26: /MGTTX2_P -> /FMC_LA03_P
- P3 pad 27: /FMC_LA00_CC_N -> /FMC_LA04_N
- P3 pad 28: /SFP_GBT_TX_P -> /FMC_LA03_N
- P3 pad 29: /FMC_LA01_CC_P -> /1V2_AVTT
- P3 pad 3: /FMC_LA14_N -> /MGTREFCLK1_N
- P3 pad 30: /MGTTX2_N -> GND
- P3 pad 31: /FMC_LA00_CC_P -> /1V2_AVTT
- P3 pad 32: /SFP_GBT_TX_N -> /FMC_LA05_P
- P3 pad 33: GND -> /SD1_B_CMD
- P3 pad 34: GND -> /FMC_LA05_N
- P3 pad 35: GND -> /SD1_B_DAT1
- P3 pad 37: /FMC_LA10_N -> /SD1_B_DAT3
- P3 pad 38: /FMC_LA02_P -> /SD1_B_DAT0
- P3 pad 39: /FMC_LA11_N -> GND
- P3 pad 4: Net-(P3-Pad2) -> Net-(P3-Pad4)
- P3 pad 40: Net-(P3-Pad20) -> /SD1_B_DAT2
- P3 pad 41: /FMC_LA10_P -> /FMC_LA06_P
- P3 pad 42: /FMC_LA02_N -> /SD1_B_CDN
- P3 pad 43: /FMC_LA11_P -> /FMC_LA06_N
- P3 pad 44: Net-(P3-Pad22) -> /SD1_B_CLK
- P3 pad 45: GND -> /VADJ
- P3 pad 46: GND -> /VADJ
- P3 pad 47: GND -> /ETH0_PHY_LED1
- P3 pad 48: GND -> /ETH0_PHY_LED0
- P3 pad 49: /FMC_LA08_N -> GND
- P3 pad 5: /FMC_LA13_P -> GND
- P3 pad 50: /FMC_LA04_P -> GND
- P3 pad 51: /FMC_LA09_N -> /ETH0_MD2_P
- P3 pad 52: /FMC_LA03_P -> /ETH0_MD1_P
- P3 pad 53: /FMC_LA08_P -> /ETH0_MD2_N
- P3 pad 54: /FMC_LA04_N -> /ETH0_MD1_N
- P3 pad 55: /FMC_LA09_P -> GND
- P3 pad 56: /FMC_LA03_N -> GND
- P3 pad 57: GND -> /ETH0_MD4_P
- P3 pad 58: /1V2_AVTT -> /ETH0_MD3_P
- P3 pad 59: GND -> /ETH0_MD4_N
- P3 pad 6: /MGTREFCLK1_N -> /1V0_AVCC
- P3 pad 60: GND -> /ETH0_MD3_N
- P3 pad 61: /FMC_LA08_N -> GND
- P3 pad 62: /1V2_AVTT -> GND
- P3 pad 63: /USB_OTG_CPEN -> /FMC_LA07_P
- P3 pad 64: /FMC_LA05_P -> /USB_OTG_ID
- P3 pad 65: /FMC_LA08_P -> /FMC_LA07_P
- P3 pad 66: /SD1_B_CMD -> GND
- P3 pad 68: /FMC_LA05_N -> /FMC_LA08_P
- P3 pad 69: GND -> /USB_OTG_CPEN
- P3 pad 7: /FMC_LA14_P -> /FMC_GBT_TX_P
- P3 pad 70: /SD1_B_DAT1 -> /FMC_LA08_N
- P3 pad 71: /FMC_LA07_P -> GND
- P3 pad 73: /USB_OTG_ID -> /FMC_LA09_P
- P3 pad 74: /SD1_B_DAT3 -> /FMC_LA08_P
- P3 pad 75: /FMC_LA07_P -> /FMC_LA09_N
- P3 pad 76: /SD1_B_DAT0 -> /FMC_LA08_N
- P3 pad 79: GND -> /FMC_LA11_P
- P3 pad 8: Net-(P3-Pad4) -> /1V0_AVCC
- P3 pad 80: /SD1_B_DAT2 -> /FMC_LA10_P
- P3 pad 81: /ETH0_MD3_N -> /FMC_LA11_N
- P3 pad 82: /FMC_LA06_P -> /FMC_LA10_N
- P3 pad 83: /ETH0_MD4_N -> GND
- P3 pad 84: /SD1_B_CDN -> GND
- P3 pad 85: /ETH0_MD3_P -> /FMC_LA00_CC_P
- P3 pad 86: /FMC_LA06_N -> /FMC_LA01_CC_P
- P3 pad 87: /ETH0_MD4_P -> /FMC_LA00_CC_N
- P3 pad 88: /SD1_B_CLK -> /FMC_LA01_CC_N
- P3 pad 9: GND -> /FMC_GBT_TX_N
- P3 pad 90: /VADJ -> GND
- P3 pad 91: GND -> /FMC_LA12_P
- P3 pad 92: /VADJ -> /FMC_CLK0_M2C_P
- P3 pad 93: /ETH0_MD1_N -> /FMC_LA12_N
- P3 pad 94: /ETH0_PHY_LED1 -> /FMC_CLK0_M2C_N
- P3 pad 95: /ETH0_MD2_N -> GND
- P3 pad 96: /ETH0_PHY_LED0 -> GND
- P3 pad 97: /ETH0_MD1_P -> /FMC_LA14_P
- P3 pad 98: GND -> /FMC_LA13_P
- P3 pad 99: /ETH0_MD2_P -> /FMC_LA14_N
- P4 pad 1: /USB_UART_RXD -> /AD9361_GPO1
- P4 pad 10: GND -> Net-(P4-Pad10)
- P4 pad 100: GND -> /USB_UART_RXD
- P4 pad 13: /SGPIO3 -> /LED_GPIO_1
- P4 pad 14: /AD9361_AUXAC1 -> /DIP_GPIO_1
- P4 pad 15: /SYS_SCL -> /LED_GPIO_2
- P4 pad 16: /AD9361_AUXADC -> /DIP_GPIO_2
- P4 pad 17: /SGPIO2 -> GND
- P4 pad 18: /AD9361_AUXAC2 -> GND
- P4 pad 19: /SYS_SDA -> /CAM_GPIO_2
- P4 pad 20: Net-(P4-Pad10) -> /CAM_GPIO_0
- P4 pad 21: GND -> /CAM_GPIO_3
- P4 pad 22: GND -> /CAM_GPIO_1
- P4 pad 25: /GPIO3 -> /CAM_GPIO_6
- P4 pad 26: /LED_GPIO_1 -> /CAM_GPIO_4
- P4 pad 27: /SGPIO1 -> /CAM_GPIO_7
- P4 pad 28: /DIP_GPIO_1 -> /CAM_GPIO_5
- P4 pad 29: /GPIO2 -> GND
- P4 pad 3: /ETH1_RESETN -> /AD9361_GPO3
- P4 pad 30: /LED_GPIO_2 -> GND
- P4 pad 31: /SGPIO0 -> /I2S_MCLK
- P4 pad 32: /DIP_GPIO_2 -> /CAM_GPIO_8
- P4 pad 33: GND -> /I2S_BCLK
- P4 pad 34: GND -> /RF_GPIO3_BANK34
- P4 pad 35: GND -> /I2S_SDATA_IN
- P4 pad 36: GND -> /I2S_LRCLK
- P4 pad 37: Net-(P4-Pad82) -> /PB_GPIO_1
- P4 pad 38: /CAM_GPIO_2 -> /I2S_SDATA_OUT
- P4 pad 39: Net-(P4-Pad81) -> GND
- P4 pad 4: /AD9361_GPO0 -> /AD9361_GPO2
- P4 pad 40: /CAM_GPIO_0 -> GND
- P4 pad 41: /SPI2_MOSI -> /ETH1_RX_CLK
- P4 pad 42: /CAM_GPIO_3 -> /PB_GPIO_2
- P4 pad 43: /GPIO1 -> /ETH1_RXD1
- P4 pad 44: /CAM_GPIO_1 -> /PB_GPIO_3
- P4 pad 45: /SPI2_SCK -> /ETH1_RX_CLK
- P4 pad 46: GND -> /ETH1_RXD2
- P4 pad 47: /GPIO0 -> /ETH1_RX_CTRL
- P4 pad 48: GND -> /ET1_RXD3
- P4 pad 49: /SYS_SPI_NSS -> GND
- P4 pad 5: Net-(P4-Pad98) -> GND
- P4 pad 50: /CAM_GPIO_6 -> GND
- P4 pad 51: /SPI2_MISO -> /ETH1_TXD0
- P4 pad 52: /CAM_GPIO_4 -> /ETH1_TX_CLK
- P4 pad 53: /SYS_SPI_MISO -> /ETH1_TXD1
- P4 pad 54: /CAM_GPIO_7 -> /ETH1_TX_CTRL
- P4 pad 55: /SPI2_NSS -> GND
- P4 pad 56: /CAM_GPIO_5 -> GND
- P4 pad 57: GND -> /ETH1_MDC
- P4 pad 58: GND -> /ETH1_TXD2
- P4 pad 59: GND -> /ETH1_MDIO
- P4 pad 6: /AD9361_GPO3 -> GND
- P4 pad 60: GND -> /EHT1_TXD3
- P4 pad 61: /LED_GPIO_0 -> GND
- P4 pad 62: /I2S_MCLK -> GND
- P4 pad 63: /FAN_TACH -> /RF_GPIO4_BANK34
- P4 pad 64: /CAM_GPIO_8 -> /AD9361_CLK
- P4 pad 65: /RF_GPIO5_BANK34 -> GND
- P4 pad 66: /I2S_BCLK -> GND
- P4 pad 68: /RF_GPIO3_BANK34 -> /RF_GPIO5_BANK34
- P4 pad 69: GND -> /FAN_TACH
- P4 pad 7: /USB_UART_TXD -> /AD9361_AUXAC1
- P4 pad 70: /I2S_SDATA_IN -> /LED_GPIO_0
- P4 pad 72: /I2S_LRCLK -> GND
- P4 pad 73: /AD9361_CLK -> /SPI2_NSS
- P4 pad 74: /PB_GPIO_1 -> /SYS_SPI_MISO
- P4 pad 75: /RF_GPIO4_BANK34 -> /SPI2_MISO
- P4 pad 76: /I2S_SDATA_OUT -> /SYS_SPI_NSS
- P4 pad 77: GND -> /GPIO0
- P4 pad 78: GND -> /SPI2_SCK
- P4 pad 79: GND -> /GPIO1
- P4 pad 8: /AD9361_GPO2 -> /AD9361_AUXADC
- P4 pad 80: GND -> /SPI2_MOSI
- P4 pad 81: /EHT1_TXD3 -> Net-(P4-Pad81)
- P4 pad 82: /ETH1_RX_CLK -> Net-(P4-Pad82)
- P4 pad 83: /ETH1_MDIO -> GND
- P4 pad 84: /PB_GPIO_2 -> GND
- P4 pad 85: /ETH1_TXD2 -> /SGPIO0
- P4 pad 86: /ETH1_RXD1 -> /GPIO2
- P4 pad 87: /ETH1_MDC -> /SGPIO1
- P4 pad 88: /PB_GPIO_3 -> /GPIO3
- P4 pad 9: GND -> /AD9361_AUXAC2
- P4 pad 90: /ETH1_RX_CLK -> GND
- P4 pad 91: GND -> /SYS_SDA
- P4 pad 92: /ETH1_RXD2 -> /SGPIO2
- P4 pad 93: /ETH1_TX_CTRL -> /SYS_SCL
- P4 pad 94: /ETH1_RX_CTRL -> /SGPIO3
- P4 pad 95: /ETH1_TXD1 -> GND
- P4 pad 96: /ET1_RXD3 -> GND
- P4 pad 97: /ETH1_TX_CLK -> /USB_UART_TXD
- P4 pad 98: GND -> Net-(P4-Pad98)
- P4 pad 99: /ETH1_TXD0 -> /ETH1_RESETN
Routing:
- net /1V2_AVTT: track 1.92 -> 0.00 mm
- net /SD1_B_CLK: track 0.00 -> 0.99 mm
- net /VADJ: track 0.93 -> 0.00 mm
- net /SD1_B_DAT2: track 0.00 -> 0.93 mm
- net /FMC_LA08_P: track 0.00 -> 0.93 mm
Other:
- board outline added: 62 x 106.9 mm
