File: payload_board.sch (KiCad schematic (older format))
At the start: 6 parts, among them P1 CONN_02X50, P2 CONN_02X50, P3 CONN_02X50, P4 CONN_02X50, P5 CONN_02X26, P6 CONN_02X26

Commit message: Add files via upload
Parts:
- added P7: CONN_02X30, Connectors_Samtec:MECF-30-0_-NP-L-DV_Edge, symbol CONN_02X30
Connections:
- net +3V3: now also P7.11 (P11), P7.14 (P14), P7.2 (P2), P7.33 (P33), P7.36 (P36), P7.53 (P53), P7.56 (P56)
- net +5V: now also P7.3 (P3), P7.57 (P57)
- net CFG_INIT__B: now also P2.10 (P10)
- net GND: now also P7.1 (P1), P7.12 (P12), P7.13 (P13), P7.16 (P16), P7.17 (P17), P7.20 (P20), P7.23 (P23), P7.26 (P26), P7.27 (P27), P7.30 (P30), P7.31 (P31), P7.34 (P34), P7.35 (P35), P7.38 (P38), P7.39 (P39), P7.4 (P4), P7.42 (P42), P7.43 (P43), P7.46 (P46), P7.47 (P47), P7.5 (P5), P7.50 (P50), P7.51 (P51), P7.54 (P54), P7.55 (P55), P7.58 (P58), P7.59 (P59), P7.8 (P8), P7.9 (P9)
- net SPI2_MISO: now also P7.15 (P15)
- net SPI2_MOSI: now also P7.18 (P18)
- net SPI2_SCK: now also P7.19 (P19)
- net SYS_SCL: now also P7.7 (P7)
- net SYS_SDA: now also P7.10 (P10)
- new net +12V: P7.6 (P6), P7.60 (P60)
- new net GPIO_10: P7.49 (P49)
- new net GPIO_11: P7.52 (P52)
- new net GPIO_7: P7.44 (P44)
- new net GPIO_8: P7.45 (P45)
- new net GPIO_9: P7.48 (P48)
- new net SGPIO_0: P7.24 (P24)
- new net SGPIO_1: P7.25 (P25)
- new net SGPIO_2: P7.28 (P28)
- new net SGPIO_3: P7.29 (P29)
- new net SGPIO_4: P7.32 (P32)
- new net SYS_MISO: P7.37 (P37)
- new net SYS_MOSI: P7.40 (P40)
- new net SYS_SCK: P7.41 (P41)
