File: breakoutBoard/_saved_payload_board.sch (KiCad schematic (older format))
At the start: 8 parts, among them J1 Conn_01x40, P1 CONN_02X50, P2 CONN_02X50, P3 CONN_02X50, P4 CONN_02X50, P5 CONN_02X26, P6 CONN_02X26, P7 CONN_02X30

Commit message: Started work on breakout board
Parts:
- added J? (x2): Conn_01x40, symbol Conn_01x40
Connections:
- net labels added: MIO48
- wire segments 561 -> 574
Other:
- note added: "JX1\n"
- note added: "JX2\n"
- note added: "JX3"
- note added: "JX4"
- moved on the sheet: P1A, P1B, P2A, P2B, P3A, P3B, P4A, P4B
