File: breakoutBoard/_saved_payload_board.sch (KiCad schematic (older format))
At the start: 10 parts, among them J1 Power_Breakout, J2 MIO_Breakout, J3 USB_OTG_Breakout, J4 Cardedge breakout, P1 CONN_02X50, P2 CONN_02X50, P3 CONN_02X50, P4 CONN_02X50, P5 CONN_02X30, P7 CONN_02X30

Commit message: Work on schematic and traces
Parts:
- J4: footprint Pin_Headers:Pin_Header_Straight_1x15_Pitch2.54mm -> Pin_Headers:Pin_Header_Straight_1x17_Pitch2.54mm
Connections:
- net MIO10: now also P5.25 (Pin_25); no longer P5.21 (Pin_21)
- net MIO11: now also P5.26 (Pin_26); no longer P5.22 (Pin_22)
- net MIO12: now also P5.30 (Pin_30); no longer P5.26 (Pin_26)
- net MIO15: now also P5.29 (Pin_29); no longer P5.25 (Pin_25)
- no-connect marks 2 -> 4
Changed lines of the file:
@@
 	1    0    0    -1
 $EndComp
+Text GLabel 14800 5700 2    60   Input ~ 0
+MIO12
 Text GLabel 14800 5500 2    60   Input ~ 0
-MIO12
-Text GLabel 14800 5300 2    60   Input ~ 0
 MIO11
 Text GLabel 14800 5100 2    60   Input ~ 0
@@
 Text GLabel 14800 4500 2    60   Input ~ 0
 MIO51
+Text GLabel 14300 5700 0    60   Input ~ 0
+MIO15
 Text GLabel 14300 5500 0    60   Input ~ 0
-MIO15
-Text GLabel 14300 5300 0    60   Input ~ 0
 MIO10
 Text GLabel 14300 5100 0    60   Input ~ 0
@@
 F 0 "J4" H 19800 6500 50  0000 C CNN
 F 1 "Cardedge breakout" H 19900 4700 50  0000 C CNN
-F 2 "Pin_Headers:Pin_Header_Straight_1x15_Pitch2.54mm" H 19800 5600 50  0001 C CNN
+F 2 "Pin_Headers:Pin_Header_Straight_1x17_Pitch2.54mm" H 19800 5600 50  0001 C CNN
 F 3 "" H 19800 5600 50  0001 C CNN
 	1    19800 5600
@@
 NoConn ~ 17300 5250
 NoConn ~ 16800 5250
+NoConn ~ 14800 5300
+NoConn ~ 14300 5300
 $EndSCHEMATC
