File: breakoutBoard/payload_board.sch (KiCad schematic (older format))
At the start: 10 parts, among them J1 Conn_01x40, P1 CONN_02X50, P2 CONN_02X50, P3 CONN_02X50, P4 CONN_02X50, P5 CONN_02X26, P6 CONN_02X26, P7 CONN_02X30

Commit message: Basic pinout done and start of routing
Parts:
- removed J1, J? (x2): Conn_01x40, symbol Conn_01x40
- removed P5, P6: CONN_02X26, Socket_Strips:Socket_Strip_Straight_2x26_Pitch2.54mm, symbol CONN_02X26
- added J?: Power_Breakout, symbol Conn_01x09
- added J?: MIO_Breakout, symbol Conn_02x06_Counter_Clockwise
- added J?: USB_OTG_Breakout, symbol Conn_02x03_Counter_Clockwise
- P7: symbol CONN_02X30 -> Conn_02x30_Counter_Clockwise
Connections:
- net labels added: IO_00_33_JX1, IO_L01_33_JX1_N, IO_L01_33_JX1_P, IO_L16_33_JX1_N, IO_L16_33_JX1_P, IO_L18_33_JX1_N, IO_L18_33_JX1_P, IO_L20_33_JX1_N, IO_L20_33_JX1_P, IO_L22_33_JX1_N, IO_L22_33_JX1_P
- net labels removed: +12V, +3.3V, 1V0_AVCC, DIP_GPIO_0, ETH0_MD1_N, ETH0_MD1_P, ETH0_MD3_N, ETH0_MD3_P, ETH0_PHY_LED0, FMC_CLK0_M2C_N, FMC_CLK0_M2C_P, FMC_LA01_CC_N, FMC_LA01_CC_P, FMC_LA03_N, FMC_LA03_P, FMC_LA05_N, FMC_LA05_P, FMC_LA08_N, FMC_LA08_P, FMC_LA10_N, FMC_LA10_P, FMC_LA13_N, FMC_LA13_P, FPGA_Done, GPIO0, GPIO1, GPIO10, GPIO11, GPIO12, GPIO13, GPIO2, GPIO3, GPIO4, GPIO5, GPIO6, GPIO7, GPIO8, GPIO9, GPIO_10, GPIO_11, GPIO_7, GPIO_8, GPIO_9, I2C2_SCL, I2C2_SDA, I2C3_SCL, I2C3_SDA, LED_GPIO_3, NBUFEN_PRI, NBUFEN_SEC, RADIO_RR, RADIO_RX, RADIO_TR, RADIO_TX, RF_GPIO2_BANK12, SD1_B_CDN, SD1_B_CLK, SD1_B_DAT0, SD1_B_DAT2, SFP_GBT_TX_N, SFP_GBT_TX_P, SFP_GPIO_0, SFP_GPIO_1, SFP_GPIO_2, SFP_GPIO_3, SFP_GPIO_4, SFP_GPIO_5, SFP_GPIO_6, SGPIO0, SGPIO1, SGPIO10, SGPIO11, SGPIO12, SGPIO13, SGPIO14, SGPIO2, SGPIO3, SGPIO4, SGPIO5, SGPIO6, SGPIO7, SGPIO8, SGPIO9, SGPIO_0, SGPIO_1, SGPIO_2, SGPIO_3, SGPIO_4, SPI2_MISO, SPI2_MOSI, SPI2_NSS, SPI2_SCK, SYS_MISO, SYS_MOSI, SYS_RESET, SYS_SCK, SYS_SCL, SYS_SDA, SYS_SPI_MISO, SYS_SPI_MOSI, SYS_SPI_SCK, SYS_SPL_NSS, USB_OTG_ID, USB_UART_RXD, USB_UART_TXD, VADJ
- wire segments 292 -> 163

Commit message: Started routing
Parts:
- J1: renamed from J?; footprint (none) -> Pin_Headers:Pin_Header_Straight_1x09_Pitch2.54mm; symbol Conn_01x09 -> Conn_01x10
- J2: renamed from J?; footprint (none) -> Pin_Headers:Pin_Header_Straight_1x12_Pitch2.54mm; symbol Conn_02x06_Counter_Clockwise -> Conn_01x12
- J3: renamed from J?; footprint (none) -> Pin_Headers:Pin_Header_Straight_1x06_Pitch2.54mm
- P7: symbol Conn_02x30_Counter_Clockwise -> Conn_02x30_Odd_Even
Connections:
- net +5V: now also P7.2 (Pin_2), P7.33 (Pin_33), P7.34 (Pin_34); no longer P7.17 (Pin_17), P7.44 (Pin_44), P7.60 (Pin_60)
- net GND: now also J1.10 (Pin_10), P7.11 (Pin_11), P7.15 (Pin_15), P7.19 (Pin_19), P7.23 (Pin_23), P7.27 (Pin_27), P7.3 (Pin_3), P7.32 (Pin_32), P7.36 (Pin_36), P7.40 (Pin_40), P7.44 (Pin_44), P7.48 (Pin_48), P7.52 (Pin_52), P7.56 (Pin_56), P7.60 (Pin_60), P7.7 (Pin_7); no longer P7.10 (Pin_10), P7.14 (Pin_14), P7.18 (Pin_18), P7.2 (Pin_2), P7.22 (Pin_22), P7.26 (Pin_26), P7.30 (Pin_30), P7.33 (Pin_33), P7.37 (Pin_37), P7.41 (Pin_41), P7.45 (Pin_45), P7.49 (Pin_49), P7.53 (Pin_53), P7.57 (Pin_57), P7.6 (Pin_6)
- net MIO0: now also J2.11 (Pin_11), P7.9 (Pin_9); no longer J2.5 (Pin_5), P7.34 (Pin_34)
- net MIO10: now also J2.8 (Pin_8), P7.21 (Pin_21); no longer J2.2 (Pin_2), P7.38 (Pin_38)
- net MIO11: now also J2.2 (Pin_2), P7.22 (Pin_22); no longer J2.11 (Pin_11), P7.56 (Pin_56)
- net MIO12: now also J2.1 (Pin_1), P7.26 (Pin_26); no longer J2.12 (Pin_12), P7.58 (Pin_58)
- net MIO13: now also J2.9 (Pin_9), P7.17 (Pin_17); no longer J2.3 (Pin_3), P7.42 (Pin_42)
- net MIO14: now also J2.10 (Pin_10), P7.13 (Pin_13); no longer J2.4 (Pin_4), P7.40 (Pin_40)
- net MIO15: now also J2.7 (Pin_7), P7.25 (Pin_25); no longer J2.1 (Pin_1), P7.46 (Pin_46)
- net MIO46: now also J2.3 (Pin_3), P7.18 (Pin_18); no longer J2.10 (Pin_10), P7.54 (Pin_54)
- net MIO47: now also J2.4 (Pin_4), P7.14 (Pin_14); no longer J2.9 (Pin_9), P7.52 (Pin_52)
- net MIO48: now also J2.12 (Pin_12), P7.5 (Pin_5); no longer J2.6 (Pin_6), P7.36 (Pin_36)
- net MIO49: now also J2.5 (Pin_5), P7.10 (Pin_10); no longer J2.8 (Pin_8), P7.50 (Pin_50)
- net MIO51: now also J2.6 (Pin_6), P7.6 (Pin_6); no longer J2.7 (Pin_7), P7.48 (Pin_48)
- net PWR_ENABLE: now also P7.57 (Pin_57); no longer P7.3 (Pin_3)
Other:
- moved on the sheet: J2
Changed lines of the file:
@@
 AD9361_GPO_VDD
 $Comp
-L GND #PWR1
+L GND #PWR01
 U 1 1 58E02281
 P 7300 6900
-F 0 "#PWR1" H 7300 6650 50  0001 C CNN
+F 0 "#PWR01" H 7300 6650 50  0001 C CNN
 F 1 "GND" H 7300 6750 50  0000 C CNN
 F 2 "" H 7300 6900 50  0000 C CNN
@@
 $EndComp
 $Comp
-L GND #PWR2
+L GND #PWR02
 U 1 1 58E022A5
 P 8000 6900
-F 0 "#PWR2" H 8000 6650 50  0001 C CNN
+F 0 "#PWR02" H 8000 6650 50  0001 C CNN
 F 1 "GND" H 8000 6750 50  0000 C CNN
 F 2 "" H 8000 6900 50  0000 C CNN
@@
 $EndComp
 $Comp
-L GND #PWR3
+L GND #PWR03
 U 1 1 58E022C9
 P 10100 6950
-F 0 "#PWR3" H 10100 6700 50  0001 C CNN
+F 0 "#PWR03" H 10100 6700 50  0001 C CNN
 F 1 "GND" H 10100 6800 50  0000 C CNN
 F 2 "" H 10100 6950 50  0000 C CNN
@@
 $EndComp
 $Comp
-L GND #PWR4
+L GND #PWR04
 U 1 1 58E022ED
 P 10800 6950
-F 0 "#PWR4" H 10800 6700 50  0001 C CNN
+F 0 "#PWR04" H 10800 6700 50  0001 C CNN
 F 1 "GND" H 10800 6800 50  0000 C CNN
 F 2 "" H 10800 6950 50  0000 C CNN
@@
 $EndComp
 $Comp
-L GND #PWR5
+L GND #PWR05
 U 1 1 58E025D1
 P 1850 6800
-F 0 "#PWR5" H 1850 6550 50  0001 C CNN
+F 0 "#PWR05" H 1850 6550 50  0001 C CNN
 F 1 "GND" H 1850 6650 50  0000 C CNN
 F 2 "" H 1850 6800 50  0000 C CNN
@@
 $EndComp
 $Comp
-L GND #PWR6
+L GND #PWR06
 U 1 1 58E025F5
 P 2550 6800
-F 0 "#PWR6" H 2550 6550 50  0001 C CNN
+F 0 "#PWR06" H 2550 6550 50  0001 C CNN
 F 1 "GND" H 2550 6650 50  0000 C CNN
 F 2 "" H 2550 6800 50  0000 C CNN
@@
 $EndComp
 $Comp
-L GND #PWR7
+L GND #PWR07
 U 1 1 58E02619
 P 4550 6900
-F 0 "#PWR7" H 4550 6650 50  0001 C CNN
+F 0 "#PWR07" H 4550 6650 50  0001 C CNN
 F 1 "GND" H 4550 6750 50  0000 C CNN
 F 2 "" H 4550 6900 50  0000 C CNN
@@
 $EndComp
 $Comp
-L GND #PWR8
+L GND #PWR08
 U 1 1 58E0263D
 P 5250 6900
-F 0 "#PWR8" H 5250 6650 50  0001 C CNN
+F 0 "#PWR08" H 5250 6650 50  0001 C CNN
 F 1 "GND" H 5250 6750 50  0000 C CNN
 F 2 "" H 5250 6900 50  0000 C CNN
@@
 JX2\n
 $Comp
-L +5V #PWR?
+L +5V #PWR09
 U 1 1 5B582995
 P 1650 4050
-F 0 "#PWR?" H 1650 3900 50  0001 C CNN
+F 0 "#PWR09" H 1650 3900 50  0001 C CNN
 F 1 "+5V" H 1650 4190 50  0000 C CNN
 F 2 "" H 1650 4050 50  0001 C CNN
@@
 $EndComp
 $Comp
-L +5V #PWR?
+L +5V #PWR010
 U 1 1 5B582C35
 P 2700 4050
-F 0 "#PWR?" H 2700 3900 50  0001 C CNN
+F 0 "#PWR010" H 2700 3900 50  0001 C CNN
 F 1 "+5V" H 2700 4190 50  0000 C CNN
 F 2 "" H 2700 4050 50  0001 C CNN
@@
 JX_VCCO_12
 $Comp
-L +5V #PWR?
+L +5V #PWR011
 U 1 1 5B583F63
 P 5400 1500
-F 0 "#PWR?" H 5400 1350 50  0001 C CNN
+F 0 "#PWR011" H 5400 1350 50  0001 C CNN
 F 1 "+5V" H 5400 1640 50  0000 C CNN
 F 2 "" H 5400 1500 50  0001 C CNN
@@
 $EndComp
 $Comp
-L +5V #PWR?
+L +5V #PWR012
 U 1 1 5B585EBB
 P 4350 4000
-F 0 "#PWR?" H 4350 3850 50  0001 C CNN
+F 0 "#PWR012" H 4350 3850 50  0001 C CNN
 F 1 "+5V" H 4350 4140 50  0000 C CNN
 F 2 "" H 4350 4000 50  0001 C CNN
@@
 $EndComp
 $Comp
-L +5V #PWR?
+L +5V #PWR013
 U 1 1 5B586104
 P 5450 4000
-F 0 "#PWR?" H 5450 3850 50  0001 C CNN
+F 0 "#PWR013" H 5450 3850 50  0001 C CNN
 F 1 "+5V" H 5450 4140 50  0000 C CNN
 F 2 "" H 5450 4000 50  0001 C CNN
@@
 IO_L01_33_JX1_N
 $Comp
-L Conn_02x30_Counter_Clockwise P7
+L Conn_02x30_Odd_Even P7
 U 1 1 5B15A0EA
 P 14550 5600
@@
 JX_MGTAVTT
 $Comp
-L +5V #PWR?
+L +5V #PWR014
 U 1 1 5B58ED6F
 P 2450 10250
-F 0 "#PWR?" H 2450 10100 50  0001 C CNN
+F 0 "#PWR014" H 2450 10100 50  0001 C CNN
 F 1 "+5V" H 2450 10390 50  0000 C CNN
 F 2 "" H 2450 10250 50  0001 C CNN
@@
 $EndComp
 $Comp
-L Conn_01x09 J?
+L Conn_01x10 J1
 U 1 1 5B58EE37
 P 2100 9850
-F 0 "J?" H 2100 10350 50  0000 C CNN
-F 1 "Power_Breakout" H 2100 9350 50  0000 C CNN
-F 2 "" H 2100 9850 50  0001 C CNN
+F 0 "J1" H 2100 10350 50  0000 C CNN
+F 1 "Power_Breakout" H 2100 9250 50  0000 C CNN
+F 2 "Pin_Headers:Pin_Header_Straight_1x09_Pitch2.54mm" H 2100 9850 50  0001 C CNN
 F 3 "" H 2100 9850 50  0001 C CNN
 	1    2100 9850
 	-1   0    0    1
 $EndComp
-Text GLabel 4600 9600 0    60   Input ~ 0
+Text GLabel 5000 10050 2    60   Input ~ 0
 MIO15
-Text GLabel 4600 9700 0    60   Input ~ 0
+Text GLabel 5000 10150 2    60   Input ~ 0
 MIO10
-Text GLabel 4600 9800 0    60   Input ~ 0
+Text GLabel 5000 10250 2    60   Input ~ 0
 MIO13
-Text GLabel 4600 9900 0    60   Input ~ 0
+Text GLabel 5000 10350 2    60   Input ~ 0
 MIO14
-Text GLabel 4600 10000 0    60   Input ~ 0
+Text GLabel 5000 10450 2    60   Input ~ 0
 MIO0
-Text GLabel 4600 10100 0    60   Input ~ 0
+Text GLabel 5000 10550 2    60   Input ~ 0
 MIO48
-Text GLabel 5100 9600 2    60   Input ~ 0
+Text GLabel 5000 9450 2    60   Input ~ 0
 MIO12
-Text GLabel 5100 9700 2    60   Input ~ 0
+Text GLabel 5000 9550 2    60   Input ~ 0
 MIO11
-Text GLabel 5100 9800 2    60   Input ~ 0
+Text GLabel 5000 9650 2    60   Input ~ 0
 MIO46
-Text GLabel 5100 9900 2    60   Input ~ 0
+Text GLabel 5000 9750 2    60   Input ~ 0
 MIO47
-Text GLabel 5100 10000 2    60   Input ~ 0
+Text GLabel 5000 9850 2    60   Input ~ 0
 MIO49
-Text GLabel 5100 10100 2    60   Input ~ 0
+Text GLabel 5000 9950 2    60   Input ~ 0
 MIO51
 $Comp
-L Conn_02x06_Counter_Clockwise J?
+L Conn_01x12 J2
 U 1 1 5B58F7D7
-P 4800 9800
-F 0 "J?" H 4850 10100 50  0000 C CNN
-F 1 "MIO_Breakout" H 4850 9400 50  0000 C CNN
-F 2 "" H 4800 9800 50  0001 C CNN
-F 3 "" H 4800 9800 50  0001 C CNN
-	1    4800 9800
-	1    0    0    -1
+P 4800 9950
+F 0 "J2" H 4800 10550 50  0000 C CNN
+F 1 "MIO_Breakout" H 4800 9250 50  0000 C CNN
+F 2 "Pin_Headers:Pin_Header_Straight_1x12_Pitch2.54mm" H 4800 9950 50  0001 C CNN
+F 3 "" H 4800 9950 50  0001 C CNN
+	1    4800 9950
+	-1   0    0    -1
 $EndComp
 Text GLabel 7950 9900 2    60   Input ~ 0
@@
 USB_OTG_N
 $Comp
-L Conn_02x03_Counter_Clockwise J?
+L Conn_02x03_Counter_Clockwise J3
 U 1 1 5B58FC0A
 P 7650 9900
-F 0 "J?" H 7700 10100 50  0000 C CNN
+F 0 "J3" H 7700 10100 50  0000 C CNN
 F 1 "USB_OTG_Breakout" H 7700 9700 50  0000 C CNN
-F 2 "" H 7650 9900 50  0001 C CNN
+F 2 "Pin_Headers:Pin_Header_Straight_1x06_Pitch2.54mm" H 7650 9900 50  0001 C CNN
 F 3 "" H 7650 9900 50  0001 C CNN
 	1    7650 9900
@@
 Wire Wire Line
 	2300 10250 2450 10250
-Wire Wire Line
-	14350 4200 14250 4200
-Wire Wire Line
-	14250 4200 14250 4050
-Wire Wire Line
-	14850 4200 14950 4200
-Wire Wire Line
-	14950 4200 14950 4050
-$Comp
-L +5V #PWR?
+$Comp
+L +5V #PWR015
 U 1 1 5B590283
 P 14950 4050
-F 0 "#PWR?" H 14950 3900 50  0001 C CNN
+F 0 "#PWR015" H 14950 3900 50  0001 C CNN
 F 1 "+5V" H 14950 4190 50  0000 C CNN
 F 2 "" H 14950 4050 50  0001 C CNN
@@
 $EndComp
 $Comp
-L +5V #PWR?
+L +5V #PWR016
 U 1 1 5B5902AF
 P 14250 4050
-F 0 "#PWR?" H 14250 3900 50  0001 C CNN
+F 0 "#PWR016" H 14250 3900 50  0001 C CNN
 F 1 "+5V" H 14250 4190 50  0000 C CNN
 F 2 "" H 14250 4050 50  0001 C CNN
@@
 	15100 4300 15100 7450
 $Comp
-L GND #PWR?
+L GND #PWR017
 U 1 1 5B5904EA
 P 15100 7450
-F 0 "#PWR?" H 15100 7200 50  0001 C CNN
+F 0 "#PWR017" H 15100 7200 50  0001 C CNN
 F 1 "GND" H 15100 7300 50  0000 C CNN
 F 2 "" H 15100 7450 50  0001 C CNN
@@
 $EndComp
 $Comp
-L GND #PWR?
+L GND #PWR018
 U 1 1 5B590516
 P 14100 7450
-F 0 "#PWR?" H 14100 7200 50  0001 C CNN
+F 0 "#PWR018" H 14100 7200 50  0001 C CNN
 F 1 "GND" H 14100 7300 50  0000 C CNN
 F 2 "" H 14100 7450 50  0001 C CNN
@@
 	1    0    0    -1
 $EndComp
+Text GLabel 14850 5400 2    60   Input ~ 0
+MIO12
+Text GLabel 14850 5200 2    60   Input ~ 0
+MIO11
+Text GLabel 14850 5000 2    60   Input ~ 0
+MIO46
+Text GLabel 14850 4800 2    60   Input ~ 0
+MIO47
+Text GLabel 14850 4600 2    60   Input ~ 0
+MIO49
 Text GLabel 14850 4400 2    60   Input ~ 0
-MIO12
-Text GLabel 14850 4600 2    60   Input ~ 0
-MIO11
-Text GLabel 14850 4800 2    60   Input ~ 0
-MIO46
-Text GLabel 14850 5000 2    60   Input ~ 0
-MIO47
-Text GLabel 14850 5200 2    60   Input ~ 0
-MIO49
-Text GLabel 14850 5400 2    60   Input ~ 0
 MIO51
-Text GLabel 14850 5600 2    60   Input ~ 0
+Text GLabel 14350 5400 0    60   Input ~ 0
 MIO15
-Text GLabel 14850 6400 2    60   Input ~ 0
+Text GLabel 14350 5200 0    60   Input ~ 0
 MIO10
-Text GLabel 14850 6000 2    60   Input ~ 0
+Text GLabel 14350 5000 0    60   Input ~ 0
 MIO13
-Text GLabel 14850 6200 2    60   Input ~ 0
+Text GLabel 14350 4800 0    60   Input ~ 0
 MIO14
-Text GLabel 14850 6800 2    60   Input ~ 0
+Text GLabel 14350 4600 0    60   Input ~ 0
 MIO0
-Text GLabel 14850 6600 2    60   Input ~ 0
+Text GLabel 14350 4400 0    60   Input ~ 0
 MIO48
 Wire Wire Line
@@
 	15400 5800 15400 5700
 $Comp
-L +5V #PWR?
+L +5V #PWR019
 U 1 1 5B592912
 P 15400 5700
-F 0 "#PWR?" H 15400 5550 50  0001 C CNN
+F 0 "#PWR019" H 15400 5550 50  0001 C CNN
 F 1 "+5V" H 15400 5840 50  0000 C CNN
 F 2 "" H 15400 5700 50  0001 C CNN
@@
 	13850 5800 13850 5700
 $Comp
-L +5V #PWR?
+L +5V #PWR020
 U 1 1 5B592A6B
 P 13850 5700
-F 0 "#PWR?" H 13850 5550 50  0001 C CNN
+F 0 "#PWR020" H 13850 5550 50  0001 C CNN
 F 1 "+5V" H 13850 5840 50  0000 C CNN
 F 2 "" H 13850 5700 50  0001 C CNN
@@
 	1    0    0    -1
 $EndComp
-Text GLabel 14350 4400 0    60   Input ~ 0
+Text GLabel 14350 7000 0    60   Input ~ 0
 PWR_ENABLE
+Wire Wire Line
+	14850 4200 14950 4200
+Wire Wire Line
+	14950 4200 14950 4050
+Wire Wire Line
+	14350 4200 14250 4200
+Wire Wire Line
+	14250 4200 14250 4050
+Wire Wire Line
+	2300 9350 2600 9350
+Wire Wire Line
+	2600 9350 2600 9200
+$Comp
+L GND #PWR?
+U 1 1 5B594135
+P 2600 9200
+F 0 "#PWR?" H 2600 8950 50  0001 C CNN
+F 1 "GND" H 2600 9050 50  0000 C CNN
+F 2 "" H 2600 9200 50  0001 C CNN
+F 3 "" H 2600 9200 50  0001 C CNN
+	1    2600 9200
+	-1   0    0    1
+$EndComp
 $EndSCHEMATC

Commit message: Work on schematic and traces
Parts:
- added J4: Cardedge breakout, Pin_Headers:Pin_Header_Straight_1x15_Pitch2.54mm, symbol Conn_01x17
- added P5: CONN_02X30, Connectors_Samtec:MECF-30-01-L-DV-WT_Socket, symbol Conn_02x30_Odd_Even
- J1: footprint Pin_Headers:Pin_Header_Straight_1x09_Pitch2.54mm -> Pin_Headers:Pin_Header_Straight_1x10_Pitch2.54mm
Connections:
- net +5V: now also P7.37 (Pin_37), P7.38 (Pin_38), J4.1 (Pin_1), P5.33 (Pin_33), P5.34 (Pin_34), P5.37 (Pin_37), P5.38 (Pin_38); no longer P7.1 (Pin_1), P7.2 (Pin_2)
- net GND: now also P1.1 (P1), P1.10 (P10), P1.100 (P100), P1.13 (P13), P1.14 (P14), P1.15 (P15), P1.16 (P16), P1.19 (P19), P1.2 (P2), P1.20 (P20), P1.21 (P21), P1.22 (P22), P1.25 (P25), P1.26 (P26), P1.27 (P27), P1.28 (P28), P1.3 (P3), P1.31 (P31), P1.33 (P33), P1.34 (P34), P1.36 (P36), P1.37 (P37), P1.38 (P38), P1.39 (P39), P1.4 (P4), P1.41 (P41), P1.42 (P42), P1.43 (P43), P1.44 (P44), P1.47 (P47), P1.48 (P48), P1.51 (P51), P1.52 (P52), P1.53 (P53), P1.54 (P54), P1.57 (P57), P1.58 (P58), P1.59 (P59), P1.60 (P60), P1.64 (P64), P1.66 (P66), P1.73 (P73), P1.74 (P74), P1.75 (P75), P1.76 (P76), P1.79 (P79), P1.8 (P8), P1.80 (P80), P1.81 (P81), P1.82 (P82), P1.85 (P85), P1.86 (P86), P1.87 (P87), P1.88 (P88), P1.91 (P91), P1.92 (P92), P1.93 (P93), P1.94 (P94), P1.97 (P97), P1.98 (P98), P1.99 (P99), P2.13 (P13), P2.14 (P14), P2.15 (P15), P2.16 (P16), P2.19 (P19), P2.20 (P20), P2.21 (P21), P2.22 (P22), P2.25 (P25), P2.26 (P26), P2.27 (P27), P2.28 (P28), P2.31 (P31), P2.32 (P32), P2.33 (P33), P2.34 (P34), P2.35 (P35), P2.36 (P36), P2.37 (P37), P2.38 (P38), P2.41 (P41), P2.42 (P42), P2.43 (P43), P2.44 (P44), P2.45 (P45), P2.46 (P46), P2.47 (P47), P2.48 (P48), P2.51 (P51), P2.52 (P52), P2.53 (P53), P2.54 (P54), P2.57 (P57), P2.58 (P58), P2.59 (P59), P2.60 (P60), P2.63 (P63), P2.64 (P64), P2.67 (P67), P2.68 (P68), P2.69 (P69), P2.70 (P70), P2.73 (P73), P2.74 (P74), P2.75 (P75), P2.76 (P76), P2.77 (P77), P2.78 (P78), P2.79 (P79), P2.80 (P80), P3.10 (P10), P3.100 (P100), P3.12 (P12), P3.14 (P14), P3.18 (P18), P3.20 (P20), P3.24 (P24), P3.26 (P26), P3.30 (P30), P3.32 (P32), P3.36 (P36), P3.38 (P38), P3.41 (P41), P3.42 (P42), P3.43 (P43), P3.44 (P44), P3.47 (P47), P3.48 (P48), P3.49 (P49), P3.50 (P50), P3.53 (P53), P3.54 (P54), P3.55 (P55), P3.56 (P56), P3.61 (P61), P3.62 (P62), P3.63 (P63), P3.64 (P64), P3.67 (P67), P3.68 (P68), P3.69 (P69), P3.70 (P70), P3.73 (P73), P3.74 (P74), P3.75 (P75), P3.76 (P76), P3.81 (P81), P3.82 (P82), P3.83 (P83), P3.84 (P84), P3.87 (P87), P3.88 (P88), P3.89 (P89), P3.90 (P90), P3.91 (P91), P3.92 (P92), P3.93 (P93), P3.94 (P94), P3.97 (P97), P3.98 (P98), P3.99 (P99), P4.1 (P1), P4.100 (P100), P4.13 (P13), P4.14 (P14), P4.17 (P17), P4.18 (P18), P4.19 (P19), P4.2 (P2), P4.20 (P20), P4.23 (P23), P4.24 (P24), P4.25 (P25), P4.26 (P26), P4.29 (P29), P4.3 (P3), P4.30 (P30), P4.31 (P31), P4.32 (P32), P4.35 (P35), P4.36 (P36), P4.37 (P37), P4.38 (P38), P4.4 (P4), P4.41 (P41), P4.42 (P42), P4.43 (P43), P4.44 (P44), P4.47 (P47), P4.48 (P48), P4.49 (P49), P4.5 (P5), P4.50 (P50), P4.53 (P53), P4.54 (P54), P4.55 (P55), P4.56 (P56), P4.6 (P6), P4.61 (P61), P4.62 (P62), P4.63 (P63), P4.64 (P64), P4.67 (P67), P4.68 (P68), P4.69 (P69), P4.7 (P7), P4.70 (P70), P4.73 (P73), P4.74 (P74), P4.75 (P75), P4.76 (P76), P4.8 (P8), P4.81 (P81), P4.82 (P82), P4.83 (P83), P4.84 (P84), P4.87 (P87), P4.88 (P88), P4.89 (P89), P4.9 (P9), P4.90 (P90), P4.93 (P93), P4.94 (P94), P4.95 (P95), P4.96 (P96), P4.97 (P97), P4.99 (P99), P7.1 (Pin_1), P7.2 (Pin_2), J4.17 (Pin_17), P5.1 (Pin_1), P5.11 (Pin_11), P5.12 (Pin_12), P5.15 (Pin_15), P5.16 (Pin_16), P5.19 (Pin_19), P5.2 (Pin_2), P5.20 (Pin_20), P5.23 (Pin_23), P5.24 (Pin_24), P5.27 (Pin_27), P5.28 (Pin_28), P5.3 (Pin_3), P5.31 (Pin_31), P5.32 (Pin_32), P5.35 (Pin_35), P5.36 (Pin_36), P5.39 (Pin_39), P5.4 (Pin_4), P5.40 (Pin_40), P5.43 (Pin_43), P5.44 (Pin_44), P5.47 (Pin_47), P5.48 (Pin_48), P5.51 (Pin_51), P5.52 (Pin_52), P5.55 (Pin_55), P5.56 (Pin_56), P5.59 (Pin_59), P5.60 (Pin_60), P5.7 (Pin_7), P5.8 (Pin_8)
- net MIO0: now also J4.9 (Pin_9), P5.9 (Pin_9)
- net MIO10: now also P7.25 (Pin_25), J4.12 (Pin_12), P5.25 (Pin_25); no longer P7.21 (Pin_21)
- net MIO11: now also P7.26 (Pin_26), J4.6 (Pin_6), P5.26 (Pin_26); no longer P7.22 (Pin_22)
- net MIO12: now also P7.30 (Pin_30), J4.7 (Pin_7), P5.30 (Pin_30); no longer P7.26 (Pin_26)
- net MIO13: now also J4.11 (Pin_11), P5.17 (Pin_17)
- net MIO14: now also J4.10 (Pin_10), P5.13 (Pin_13)
- net MIO15: now also P7.29 (Pin_29), J4.13 (Pin_13), P5.29 (Pin_29); no longer P7.25 (Pin_25)
- net MIO46: now also J4.5 (Pin_5), P5.18 (Pin_18)
- net MIO47: now also J4.4 (Pin_4), P5.14 (Pin_14)
- net MIO48: now also J4.8 (Pin_8), P5.5 (Pin_5)
- net MIO49: now also J4.3 (Pin_3), P5.10 (Pin_10)
- net MIO51: now also J4.2 (Pin_2), P5.6 (Pin_6)
- net PWR_ENABLE: now also J4.14 (Pin_14), P5.57 (Pin_57)
- net AUXDAC2: now reaches P2.10 (P10)
- net AUXADC: now reaches P2.7 (P7)
- net AUXDAC1: now reaches P2.8 (P8)
- net VDDA_GPO_PWR: now reaches P2.9 (P9)
- net FPGA_DONE: now reaches P3.8 (P8)
- net FPGA_DONE: now also P7.58 (Pin_58), J4.16 (Pin_16), P5.58 (Pin_58)
- net PG_1P8V: now reaches P4.10 (P10)
- net PG_MODULE: now reaches P4.11 (P11)
- net PG_MODULE: now also P7.53 (Pin_53), J4.15 (Pin_15), P5.53 (Pin_53)
- no-connect marks 0 -> 4
Other:
- note added: "<-Might need to remove"
- moved on the sheet: P7

Commit message: Work on schematic and traces
Parts:
- J4: footprint Pin_Headers:Pin_Header_Straight_1x15_Pitch2.54mm -> Pin_Headers:Pin_Header_Straight_1x17_Pitch2.54mm
Changed lines of the file:
@@
 F 0 "J4" H 19800 6500 50  0000 C CNN
 F 1 "Cardedge breakout" H 19900 4700 50  0000 C CNN
-F 2 "Pin_Headers:Pin_Header_Straight_1x15_Pitch2.54mm" H 19800 5600 50  0001 C CNN
+F 2 "Pin_Headers:Pin_Header_Straight_1x17_Pitch2.54mm" H 19800 5600 50  0001 C CNN
 F 3 "" H 19800 5600 50  0001 C CNN
 	1    19800 5600

Commit message: Completed routing and added gerber
Connections:
- net GND: now also J3.4 (Pin_4)
- net JX_MGTAVCC: now also J1.9 (Pin_9); no longer J1.8 (Pin_8)
- net JX_MGTAVTT: now also J1.8 (Pin_8); no longer J1.9 (Pin_9)
- net USB_OTG_CPEN: now also J3.6 (Pin_6); no longer J3.4 (Pin_4)
Changed lines of the file:
@@
 LIBS:valves
 LIBS:project
+LIBS:payload_board-cache
 EELAYER 25 0
 EELAYER END
@@
 Text GLabel 2300 9650 2    60   Input ~ 0
 3V3_I2C
+Text GLabel 2300 9450 2    60   Input ~ 0
+JX_MGTAVCC
 Text GLabel 2300 9550 2    60   Input ~ 0
-JX_MGTAVCC
-Text GLabel 2300 9450 2    60   Input ~ 0
 JX_MGTAVTT
 $Comp
@@
 Text GLabel 7950 9900 2    60   Input ~ 0
 USB_VBUS_OTG
-Text GLabel 7950 10000 2    60   Input ~ 0
+Text GLabel 7950 9800 2    60   Input ~ 0
 USB_OTG_CPEN
 Text GLabel 7450 9800 0    60   Input ~ 0
@@
 P 7650 9900
 F 0 "J3" H 7700 10100 50  0000 C CNN
-F 1 "USB_OTG_Breakout" H 7700 9700 50  0000 C CNN
+F 1 "USB_OTG_Breakout" H 7500 9650 50  0000 C CNN
 F 2 "Pin_Headers:Pin_Header_Straight_1x06_Pitch2.54mm" H 7650 9900 50  0001 C CNN
 F 3 "" H 7650 9900 50  0001 C CNN
@@
 NoConn ~ 14800 5300
 NoConn ~ 14300 5300
+$Comp
+L GND #PWR?
+U 1 1 5B5A3ACB
+P 7950 10000
+F 0 "#PWR?" H 7950 9750 50  0001 C CNN
+F 1 "GND" H 7950 9850 50  0000 C CNN
+F 2 "" H 7950 10000 50  0001 C CNN
+F 3 "" H 7950 10000 50  0001 C CNN
+	1    7950 10000
+	1    0    0    -1
+$EndComp
 $EndSCHEMATC
