File: schematics/breakoutBoard/payload_board.sch (KiCad schematic (older format))
At the start: 5 parts, among them P1 CONN_02X50, P2 CONN_02X50, P3 CONN_02X50, P4 CONN_02X50

Commit message: some fixes
Connections:
- net 3V is gone; now on net 5V: P1.57 (P57), P1.58 (P58), P1.59 (P59), P1.60 (P60), P2.12 (P12), P2.57 (P57), P2.58 (P58), P2.59 (P59), P2.60 (P60), e1.2 (5V_PWR)
- net RFGND: now reaches e1.3 (RFGND)
Changed lines of the file:
@@
 NoConn ~ 3400 7650
 NoConn ~ 1750 7050
-Text GLabel 1650 6900 2    50   Input ~ 0
-3V
+Text GLabel 1650 6900 0    50   Input ~ 0
+5V
 Text GLabel 2150 6950 2    50   Input ~ 0
 RX
-Text GLabel 2050 6850 1    50   Input ~ 0
+Text GLabel 2050 6850 1    50   Output ~ 0
 TX
-Text GLabel 1850 6700 0    50   Input ~ 0
+Text GLabel 1850 6700 2    50   Input ~ 0
 EN
+Wire Wire Line
+	1750 7050 1750 6900
+Text GLabel 1750 6900 1    50   UnSpc ~ 0
+RFGND
 $EndSCHEMATC
