File: schematics/breakoutBoard/LNA.sch (KiCad schematic (older format))
At the start: 8 parts, among them U1 CBP, U2 TAMP, U3 CBP, U4 TAMP, U5 LAT-3, U6 TAMP

Commit message: Updated schematic
Cleaned up wires and re-did labels. Added additional grounds and verified pwr, TX and RX. Reference to Issues #1, #2, #3 and #5.
Connections:
- net GND1: no longer U3.15 (GND), U3.7 (GND)
- new net: U3.15 (GND), U3.7 (GND)
Changed lines of the file:
@@
 	0    -1   -1   0
 $EndComp
-Wire Wire Line
-	1550 1900 2100 1900
 $Comp
 L power:GND1 #RFGND01
@@
 	3300 3000 3300 3150
 Connection ~ 3300 3000
-Wire Wire Line
-	4550 2350 4550 2400
-Connection ~ 4550 2400
-Wire Wire Line
-	4550 2400 4550 3000
 Connection ~ 4550 3000
 Wire Wire Line
@@
 	3400 1600 3400 1350
 Wire Wire Line
-	3400 1350 5550 1350
-Wire Wire Line
-	7850 1350 7850 1700
-Wire Wire Line
-	5550 1700 5550 1350
-Connection ~ 5550 1350
-Wire Wire Line
-	5550 1350 7850 1350
-Wire Wire Line
 	3300 3000 4550 3000
 Wire Wire Line
 	4550 3000 6700 3000
-Text GLabel 5550 1350 1    50   Input ~ 0
-5V
 Wire Wire Line
 	3400 2400 3400 2700
@@
 Wire Wire Line
 	5550 2700 7850 2700
-Text GLabel 5550 2700 3    50   Input ~ 0
-GND
 Wire Wire Line
 	8850 2100 8400 2100
@@
 Text GLabel 3100 3000 3    50   Input ~ 0
 RFGND
-Text GLabel 1850 1900 1    50   Input ~ 0
+Wire Wire Line
+	1550 1900 2100 1900
+Text Label 1800 1900 0    50   ~ 0
 RF_SIG
+Wire Wire Line
+	4550 2350 4550 3000
+Wire Wire Line
+	3400 1350 5550 1350
+Wire Wire Line
+	5550 1700 5550 1350
+Text Label 4150 1350 0    50   ~ 0
+5V
+Wire Wire Line
+	7850 1700 7850 1350
+Wire Wire Line
+	7850 1350 5550 1350
+Connection ~ 5550 1350
+Text GLabel 5150 1350 1    50   Input ~ 0
+5V
+Text GLabel 5050 2700 1    50   Input ~ 0
+GND
 $EndSCHEMATC

Commit message: Added power filter
Parts:
- added C?: CP1, symbol Device:CP1
- added L?: L, symbol Device:L
Connections:
- net 5V: now also C?.1, L?.1
- net GND: now also C?.2, L?.2
Changed lines of the file:
@@
 Text GLabel 5050 2700 1    50   Input ~ 0
 GND
+$Comp
+L Device:L L?
+U 1 1 6194A367
+P 2750 4900
+F 0 "L?" H 2803 4946 50  0000 L CNN
+F 1 "L" H 2803 4855 50  0000 L CNN
+F 2 "" H 2750 4900 50  0001 C CNN
+F 3 "~" H 2750 4900 50  0001 C CNN
+	1    2750 4900
+	1    0    0    -1
+$EndComp
+$Comp
+L Device:CP1 C?
+U 1 1 6194A9C4
+P 2250 4900
+F 0 "C?" H 2365 4946 50  0000 L CNN
+F 1 "CP1" H 2365 4855 50  0000 L CNN
+F 2 "" H 2250 4900 50  0001 C CNN
+F 3 "~" H 2250 4900 50  0001 C CNN
+	1    2250 4900
+	1    0    0    -1
+$EndComp
+Wire Wire Line
+	2250 4750 2750 4750
+Wire Wire Line
+	2250 5050 2750 5050
+Text GLabel 2500 5050 3    50   Input ~ 0
+GND
+Text GLabel 2500 4750 1    50   Input ~ 0
+5V
 $EndSCHEMATC
