File: schematics/breakoutBoard/LNA.kicad_sch (KiCad schematic)
At the start: 8 parts

Commit message: Update
Parts:
- SMA1, SMA2: value (none) -> Molex-MMCX-SMD; footprint (none) -> breakoutBoard:Molex MMCX SMD 50Ohm
- U1, U3: value (none) -> CBP; footprint (none) -> mini-circuits:CBP
- U2, U4, U6: value (none) -> TAMP; footprint (none) -> mini-circuits:MCL
- U5: value (none) -> LAT-3; footprint (none) -> RF_Mini-Circuits:Mini-Circuits_MMM168_LandPatternPL-225
Changed lines of the file:
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@@
     (in_bom yes) (on_board yes)
     (property "Reference" "U5" (id 0) (at 175.26 42.7482 0))
-    (property "Value" "" (id 1) (at 175.26 45.0596 0))
-    (property "Footprint" "" (id 2) (at 175.26 64.77 0)
+    (property "Value" "LAT-3" (id 1) (at 175.26 45.0596 0))
+    (property "Footprint" "RF_Mini-Circuits:Mini-Circuits_MMM168_LandPatternPL-225" (id 2) (at 175.26 64.77 0)
       (effects (font (size 1.27 1.27)) hide)
     )
@@
       (effects (font (size 1.27 1.27)) (justify left))
     )
-    (property "Value" "" (id 1) (at 101.4476 51.943 0)
+    (property "Value" "TAMP" (id 1) (at 101.4476 51.943 0)
       (effects (font (size 1.27 1.27)) (justify left))
     )
-    (property "Footprint" "" (id 2) (at 87.63 50.8 0)
+    (property "Footprint" "mini-circuits:MCL" (id 2) (at 87.63 50.8 0)
       (effects (font (size 1.27 1.27)) hide)
     )
@@
       (effects (font (size 1.27 1.27)) (justify left))
     )
-    (property "Value" "" (id 1) (at 156.0576 54.483 0)
+    (property "Value" "TAMP" (id 1) (at 156.0576 54.483 0)
       (effects (font (size 1.27 1.27)) (justify left))
     )
-    (property "Footprint" "" (id 2) (at 142.24 53.34 0)
+    (property "Footprint" "mini-circuits:MCL" (id 2) (at 142.24 53.34 0)
       (effects (font (size 1.27 1.27)) hide)
     )
@@
       (effects (font (size 1.27 1.27)) (justify left))
     )
-    (property "Value" "" (id 1) (at 214.4776 54.483 0)
+    (property "Value" "TAMP" (id 1) (at 214.4776 54.483 0)
       (effects (font (size 1.27 1.27)) (justify left))
     )
-    (property "Footprint" "" (id 2) (at 200.66 53.34 0)
+    (property "Footprint" "mini-circuits:MCL" (id 2) (at 200.66 53.34 0)
       (effects (font (size 1.27 1.27)) hide)
     )
@@
     (in_bom yes) (on_board yes)
     (property "Reference" "U1" (id 0) (at 60.96 40.259 0))
-    (property "Value" "" (id 1) (at 60.96 42.5704 0))
-    (property "Footprint" "" (id 2) (at 60.96 49.53 0)
+    (property "Value" "CBP" (id 1) (at 60.96 42.5704 0))
+    (property "Footprint" "mini-circuits:CBP" (id 2) (at 60.96 49.53 0)
       (effects (font (size 1.27 1.27)) hide)
     )
@@
     (in_bom yes) (on_board yes)
     (property "Reference" "U3" (id 0) (at 119.38 42.799 0))
-    (property "Value" "" (id 1) (at 119.38 45.1104 0))
-    (property "Footprint" "" (id 2) (at 119.38 52.07 0)
+    (property "Value" "CBP" (id 1) (at 119.38 45.1104 0))
+    (property "Footprint" "mini-circuits:CBP" (id 2) (at 119.38 52.07 0)
       (effects (font (size 1.27 1.27)) hide)
     )
@@
     (in_bom yes) (on_board yes)
     (property "Reference" "SMA1" (id 0) (at 32.6898 44.8818 90))
-    (property "Value" "" (id 1) (at 43.18 48.26 0)
+    (property "Value" "Molex-MMCX-SMD" (id 1) (at 43.18 48.26 0)
       (effects (font (size 1.27 1.27)) hide)
     )
-    (property "Footprint" "" (id 2) (at 33.02 48.26 0)
+    (property "Footprint" "breakoutBoard:Molex MMCX SMD 50Ohm" (id 2) (at 33.02 48.26 0)
       (effects (font (size 1.27 1.27)) hide)
     )
@@
       (effects (font (size 1.27 1.27)) (justify right))
     )
-    (property "Value" "" (id 1) (at 220.98 53.34 0)
+    (property "Value" "Molex-MMCX-SMD" (id 1) (at 220.98 53.34 0)
       (effects (font (size 1.27 1.27)) hide)
     )
-    (property "Footprint" "" (id 2) (at 231.14 53.34 0)
+    (property "Footprint" "breakoutBoard:Molex MMCX SMD 50Ohm" (id 2) (at 231.14 53.34 0)
       (effects (font (size 1.27 1.27)) hide)
     )
@@
       (effects (font (size 1.27 1.27)) (justify left))
     )
-    (property "Value" "" (id 1) (at 86.0552 82.0928 0)
+    (property "Value" "GND1" (id 1) (at 86.0552 82.0928 0)
       (effects (font (size 1.27 1.27)) (justify left))
     )

Commit message: Fixed grounding issue
Connections:
- net GND1: now also U1.15 (GND), U1.7 (GND), U3.15 (GND), U3.7 (GND)
Changed lines of the file:
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@@
     (pin "4")
   )
-  (symbol (lib_id "mini-circuits:TAMP") (at 87.63 50.8 0) (unit 1)
+  (symbol (lib_name "TAMP_1") (lib_id "mini-circuits:TAMP") (at 87.63 50.8 0) (unit 1)
     (in_bom yes) (on_board yes)
     (property "Reference" "U2" (id 0) (at 101.4476 49.6316 0)
@@
     (pin "10")
     (pin "11")
+    (pin "12")
     (pin "2")
     (pin "3")
@@
     (pin "9")
   )
-  (symbol (lib_id "mini-circuits:TAMP") (at 142.24 53.34 0) (unit 1)
+  (symbol (lib_name "TAMP_2") (lib_id "mini-circuits:TAMP") (at 142.24 53.34 0) (unit 1)
     (in_bom yes) (on_board yes)
     (property "Reference" "U4" (id 0) (at 156.0576 52.1716 0)
@@
     (pin "10")
     (pin "11")
+    (pin "12")
     (pin "2")
     (pin "3")
@@
     (pin "10")
     (pin "11")
+    (pin "12")
     (pin "2")
     (pin "3")
@@
     (pin "9")
   )
-  (symbol (lib_id "mini-circuits:CBP") (at 60.96 49.53 0) (unit 1)
+  (symbol (lib_name "CBP_1") (lib_id "mini-circuits:CBP") (at 60.96 49.53 0) (unit 1)
     (in_bom yes) (on_board yes)
     (property "Reference" "U1" (id 0) (at 60.96 40.259 0))
     (property "Value" "CBP" (id 1) (at 60.96 42.5704 0))
-    (property "Footprint" "mini-circuits:CBP" (id 2) (at 60.96 49.53 0)
+    (property "Footprint" "mini-circuits:CBP" (id 2) (at 60.96 45.72 0)
       (effects (font (size 1.27 1.27)) hide)
     )
