File: schematics/breakoutBoard/payload_board.kicad_sch (KiCad schematic)
At the start: 5 parts

Commit message: Update
Parts:
- P1, P2, P3, P4: value (none) -> CONN_02X50; footprint (none) -> breakoutBoard:BERGSTAK_100_PIN1_RIGHT
- e1: value (none) -> ribbon2.54mmPitch; footprint (none) -> Connector_PinHeader_2.54mm:PinHeader_1x07_P2.54mm_Vertical
Changed lines of the file:
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@@
     (in_bom yes) (on_board yes)
     (property "Reference" "P1" (id 0) (at 45.72 18.669 0))
-    (property "Value" "" (id 1) (at 45.72 20.9804 0))
-    (property "Footprint" "" (id 2) (at 45.72 73.66 0)
+    (property "Value" "CONN_02X50" (id 1) (at 45.72 20.9804 0))
+    (property "Footprint" "breakoutBoard:BERGSTAK_100_PIN1_RIGHT" (id 2) (at 45.72 73.66 0)
       (effects (font (size 1.27 1.27)) hide)
     )
@@
     (in_bom yes) (on_board yes)
     (property "Reference" "P2" (id 0) (at 110.49 19.939 0))
-    (property "Value" "" (id 1) (at 110.49 22.2504 0))
-    (property "Footprint" "" (id 2) (at 110.49 74.93 0)
+    (property "Value" "CONN_02X50" (id 1) (at 110.49 22.2504 0))
+    (property "Footprint" "breakoutBoard:BERGSTAK_100_PIN1_RIGHT" (id 2) (at 110.49 74.93 0)
       (effects (font (size 1.27 1.27)) hide)
     )
@@
     (in_bom yes) (on_board yes)
     (property "Reference" "P3" (id 0) (at 187.96 22.479 0))
-    (property "Value" "" (id 1) (at 187.96 24.7904 0))
-    (property "Footprint" "" (id 2) (at 187.96 77.47 0)
+    (property "Value" "CONN_02X50" (id 1) (at 187.96 24.7904 0))
+    (property "Footprint" "breakoutBoard:BERGSTAK_100_PIN1_RIGHT" (id 2) (at 187.96 77.47 0)
       (effects (font (size 1.27 1.27)) hide)
     )
@@
     (in_bom yes) (on_board yes)
     (property "Reference" "P4" (id 0) (at 241.3 19.939 0))
-    (property "Value" "" (id 1) (at 241.3 22.2504 0))
-    (property "Footprint" "" (id 2) (at 241.3 74.93 0)
+    (property "Value" "CONN_02X50" (id 1) (at 241.3 22.2504 0))
+    (property "Footprint" "breakoutBoard:BERGSTAK_100_PIN1_RIGHT" (id 2) (at 241.3 74.93 0)
       (effects (font (size 1.27 1.27)) hide)
     )
@@
     (in_bom yes) (on_board yes)
     (property "Reference" "P1" (id 0) (at 45.72 92.329 0))
-    (property "Value" "" (id 1) (at 45.72 94.6404 0))
-    (property "Footprint" "" (id 2) (at 45.72 147.32 0)
+    (property "Value" "CONN_02X50" (id 1) (at 45.72 94.6404 0))
+    (property "Footprint" "breakoutBoard:BERGSTAK_100_PIN1_RIGHT" (id 2) (at 45.72 147.32 0)
       (effects (font (size 1.27 1.27)) hide)
     )
@@
     (in_bom yes) (on_board yes)
     (property "Reference" "P2" (id 0) (at 111.76 94.869 0))
-    (property "Value" "" (id 1) (at 111.76 97.1804 0))
-    (property "Footprint" "" (id 2) (at 111.76 149.86 0)
+    (property "Value" "CONN_02X50" (id 1) (at 111.76 97.1804 0))
+    (property "Footprint" "breakoutBoard:BERGSTAK_100_PIN1_RIGHT" (id 2) (at 111.76 149.86 0)
       (effects (font (size 1.27 1.27)) hide)
     )
@@
     (in_bom yes) (on_board yes)
     (property "Reference" "P3" (id 0) (at 187.96 96.139 0))
-    (property "Value" "" (id 1) (at 187.96 98.4504 0))
-    (property "Footprint" "" (id 2) (at 187.96 151.13 0)
+    (property "Value" "CONN_02X50" (id 1) (at 187.96 98.4504 0))
+    (property "Footprint" "breakoutBoard:BERGSTAK_100_PIN1_RIGHT" (id 2) (at 187.96 151.13 0)
       (effects (font (size 1.27 1.27)) hide)
     )
@@
     (in_bom yes) (on_board yes)
     (property "Reference" "P4" (id 0) (at 241.3 96.139 0))
-    (property "Value" "" (id 1) (at 241.3 98.4504 0))
-    (property "Footprint" "" (id 2) (at 241.3 151.13 0)
+    (property "Value" "CONN_02X50" (id 1) (at 241.3 98.4504 0))
+    (property "Footprint" "breakoutBoard:BERGSTAK_100_PIN1_RIGHT" (id 2) (at 241.3 151.13 0)
       (effects (font (size 1.27 1.27)) hide)
     )
@@
       (effects (font (size 1.27 1.27)) hide)
     )
-    (property "Value" "" (id 1) (at 56.5912 185.0898 0)
+    (property "Value" "ribbon2.54mmPitch" (id 1) (at 56.5912 185.0898 0)
       (effects (font (size 1.27 1.27)) (justify left))
     )
-    (property "Footprint" "" (id 2) (at 54.61 184.15 0)
-      (effects (font (size 1.27 1.27)) hide)
-    )
+    (property "Footprint" "Connector_PinHeader_2.54mm:PinHeader_1x07_P2.54mm_Vertical" (id 2) (at 54.61 184.15 0)
+      (effects (font (size 1.27 1.27)) hide)
+    )
